File: PCB/keyboard.kicad_pcb (KiCad board)
At the start: 2 copper layers, 57.2 x 78.6 mm, 30 parts, among them SW1 SW_Push, SW11 RotaryEncoder, SW2 SW_Push, SW3 SW_Push, SW4 SW_Push, SW5 SW_Push, SW6 SW_Push, SW7 SW_Push, SW8 SW_Push, SW9 SW_Push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

Commit message: mark
Other:
- board text added: "XIAO HERE"
- board text added: "Yusuf's Macropad"
Changed lines of the file:
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@@
 		(layer "Edge.Cuts")
+	)
+	(gr_text "Yusuf's Macropad"
+		(at 76.2 16.66875 0)
+		(layer "F.SilkS")
+		(effects
+			(font
+				(size 1 1)
+				(thickness 0.1)
+			)
+			(justify left bottom)
+		)
+	)
+	(gr_text "XIAO HERE"
+		(at 95.25 30.95625 0)
+		(layer "F.SilkS")
+		(effects
+			(font
+				(size 1 1)
+				(thickness 0.1)
+			)
+			(justify left bottom)
+		)
 	)
 	(segment
